Commit message: gazebo gravity fix

File: urdf/chitlits_trial.urdf (robot description, URDF)
Before this commit: robot chitlits_trial, 8 links, 7 joints
Joints:
- joint joint1: limit lower=0 upper=6.283185307179586232 effort=10000 velocity=20 -> lower=0 upper=6.283185307179586232 effort=1000000 velocity=0.5
- joint joint2: limit lower=-1.570796326794896558 upper=3.141592653589793116 effort=1000000 velocity=20 -> lower=-1.570796326794896558 upper=3.141592653589793116 effort=1000000 velocity=0.5
- joint joint3: limit lower=0 upper=6.283185307179586232 effort=100000000 velocity=20 -> lower=0 upper=6.283185307179586232 effort=1000000 velocity=0.5
- joint joint4: limit lower=0 upper=6.283185307179586232 effort=100 velocity=20 -> lower=0 upper=6.283185307179586232 effort=10000 velocity=0.5
- joint joint5: limit lower=-1.570796326794896558 upper=1.570796326794896558 effort=10 velocity=20 -> lower=-1.570796326794896558 upper=1.570796326794896558 effort=10000 velocity=0.5
- joint joint6: limit lower=0 upper=6.283185307179586232 effort=10 velocity=20 -> lower=0 upper=6.283185307179586232 effort=10000 velocity=0.5

Commit message: Increased Friction and Effort in URDF

File: urdf/chitlits_trial.urdf (robot description, URDF)
Before this commit: robot chitlits_trial, 8 links, 7 joints
Joints:
- joint joint2: limit lower=-1.570796326794896558 upper=3.141592653589793116 effort=1000000 velocity=0.5 -> lower=-1.570796326794896558 upper=3.141592653589793116 effort=2000000 velocity=0.5
- joint joint4: limit lower=0 upper=6.283185307179586232 effort=10000 velocity=0.5 -> lower=0 upper=6.283185307179586232 effort=20000 velocity=0.5
- joint joint5: limit lower=-1.570796326794896558 upper=1.570796326794896558 effort=10000 velocity=0.5 -> lower=-1.570796326794896558 upper=1.570796326794896558 effort=20000 velocity=0.5
- joint joint6: limit lower=0 upper=6.283185307179586232 effort=10000 velocity=0.5 -> lower=0 upper=6.283185307179586232 effort=20000 velocity=0.5

Commit message: i dont even remember ;-;

File: urdf/chitlits_trial.urdf (robot description, URDF)
Before this commit: robot chitlits_trial, 8 links, 7 joints
Links:
- removed link dummy_link
- added link world
Joints:
- joint dummy_joint: parent dummy_link -> world
- joint joint1: limit lower=0 upper=6.283185307179586232 effort=1000000 velocity=0.5 -> lower=-3.141592653589793116 upper=3.141592653589793116 effort=1000000 velocity=0.5
- joint joint3: limit lower=0 upper=6.283185307179586232 effort=1000000 velocity=0.5 -> lower=-3.141592653589793116 upper=3.141592653589793116 effort=1000000 velocity=0.5
- joint joint4: limit lower=0 upper=6.283185307179586232 effort=20000 velocity=0.5 -> lower=-3.141592653589793116 upper=3.141592653589793116 effort=20000 velocity=0.5
- joint joint6: limit lower=0 upper=6.283185307179586232 effort=20000 velocity=0.5 -> lower=-3.141592653589793116 upper=3.141592653589793116 effort=20000 velocity=0.5
